File: Hardware/Qwiic-Step.sch (EAGLE design)
At the start: 59 parts, among them J1 PTH, J2 Qwiic Right Angle, J3 5.5x2.1mm Barrel, J4 Qwiic Right Angle, J5 ISP, U1 A4988ALT1, U2 ATMEGA328P_TQFP, Y1 16MHz

Commit message: All traces routed, READY FOR BOARD REVIEW (other than some minor silk updates that I'll do tomorrow morning).
Parts:
- removed R6: 300k, SparkFun-Resistors:300KOHM-0603-1/10W-1%
- added R9: 22k, SparkFun-Resistors:22KOHM-0603-1/10W-1%
Connections:
- new net N$6: JP2.1, U2.ADC7
- net AMP_CUR_SENSE: now also R9.2; no longer R6.2
- net MOSI: no longer JP2.1
- net N$2: now also R9.1; no longer R6.1
Other:
- moved on the sheet: JP2
Changed lines of the file:
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@@
 <part name="SUPPLY2" library="SparkFun-PowerSymbols" deviceset="VIN" device=""/>
 <part name="U$44" library="SparkFun-IC-Amplifiers" deviceset="OPA344" device="" value="OPA344"/>
-<part name="R6" library="SparkFun-Resistors" deviceset="300KOHM" device="-0603-1/10W-1%" value="300k"/>
 <part name="R7" library="SparkFun-Resistors" deviceset="1KOHM" device="-0603-1/10W-1%" value="1k"/>
 <part name="GND21" library="SparkFun-PowerSymbols" deviceset="GND" device=""/>
+<part name="R9" library="SparkFun-Resistors" deviceset="22KOHM" device="-0603-1/10W-1%" value="22k"/>
 </parts>
 <sheets>
@@
 <attribute name="VALUE" x="147.32" y="160.274" size="1.778" layer="96" align="bottom-center"/>
 </instance>
-<instance part="GND20" gate="1" x="228.6" y="71.12" smashed="yes">
-<attribute name="VALUE" x="228.6" y="70.866" size="1.778" layer="96" align="top-center"/>
+<instance part="GND20" gate="1" x="233.68" y="106.68" smashed="yes">
+<attribute name="VALUE" x="233.68" y="106.426" size="1.778" layer="96" align="top-center"/>
 </instance>
 <instance part="SUPPLY23" gate="G$1" x="144.78" y="88.9" smashed="yes">
@@
 <attribute name="VALUE" x="34.544" y="76.581" size="1.778" layer="96" font="vector"/>
 </instance>
-<instance part="JP2" gate="G$1" x="228.6" y="81.28" smashed="yes" rot="MR270">
-<attribute name="NAME" x="226.06" y="83.82" size="1.778" layer="95" font="vector" rot="MR270"/>
-<attribute name="VALUE" x="231.14" y="83.82" size="1.778" layer="96" font="vector" rot="MR270" align="top-left"/>
+<instance part="JP2" gate="G$1" x="233.68" y="116.84" smashed="yes" rot="MR270">
+<attribute name="NAME" x="231.14" y="119.38" size="1.778" layer="95" font="vector" rot="MR270"/>
+<attribute name="VALUE" x="236.22" y="119.38" size="1.778" layer="96" font="vector" rot="MR270" align="top-left"/>
 </instance>
 <instance part="D5" gate="G$1" x="55.88" y="15.24" smashed="yes">
@@
 <attribute name="VALUE" x="-53.34" y="104.14" size="1.778" layer="95" font="vector"/>
 </instance>
-<instance part="R6" gate="G$1" x="-48.26" y="124.46" smashed="yes">
-<attribute name="NAME" x="-48.26" y="125.984" size="1.778" layer="95" font="vector" align="bottom-center"/>
-<attribute name="VALUE" x="-48.26" y="122.936" size="1.778" layer="96" font="vector" align="top-center"/>
-</instance>
 <instance part="R7" gate="G$1" x="-58.42" y="132.08" smashed="yes" rot="R90">
 <attribute name="NAME" x="-59.944" y="132.08" size="1.778" layer="95" font="vector" rot="R90" align="bottom-center"/>
@@
 <instance part="GND21" gate="1" x="-58.42" y="142.24" smashed="yes" rot="R180">
 <attribute name="VALUE" x="-58.42" y="142.494" size="1.778" layer="96" rot="R180" align="top-center"/>
+</instance>
+<instance part="R9" gate="G$1" x="-48.26" y="124.46" smashed="yes">
+<attribute name="NAME" x="-48.26" y="125.984" size="1.778" layer="95" font="vector" align="bottom-center"/>
+<attribute name="VALUE" x="-48.26" y="122.936" size="1.778" layer="96" font="vector" align="top-center"/>
 </instance>
 </instances>
@@
 </segment>
 <segment>
-<pinref part="GND20" gate="1" pin="GND"/>
-<pinref part="JP2" gate="G$1" pin="2"/>
-<wire x1="228.6" y1="73.66" x2="228.6" y2="76.2" width="0.1524" layer="91"/>
-</segment>
-<segment>
 <pinref part="R7" gate="G$1" pin="2"/>
 <wire x1="-58.42" y1="137.16" x2="-58.42" y2="139.7" width="0.1524" layer="91"/>
 <pinref part="GND21" gate="1" pin="GND"/>
+</segment>
+<segment>
+<pinref part="JP2" gate="G$1" pin="2"/>
+<pinref part="GND20" gate="1" pin="GND"/>
+<wire x1="233.68" y1="111.76" x2="233.68" y2="109.22" width="0.1524" layer="91"/>
 </segment>
 </net>
@@
 <segment>
 <pinref part="U2" gate="U1" pin="PB3(MOSI/OC2)"/>
-<wire x1="210.82" y1="88.9" x2="228.6" y2="88.9" width="0.1524" layer="91"/>
-<label x="233.68" y="88.9" size="1.27" layer="95" xref="yes"/>
-<pinref part="JP2" gate="G$1" pin="1"/>
-<wire x1="228.6" y1="88.9" x2="233.68" y2="88.9" width="0.1524" layer="91"/>
-<wire x1="228.6" y1="86.36" x2="228.6" y2="88.9" width="0.1524" layer="91"/>
-<junction x="228.6" y="88.9"/>
+<wire x1="210.82" y1="88.9" x2="213.36" y2="88.9" width="0.1524" layer="91"/>
+<label x="213.36" y="88.9" size="1.27" layer="95" xref="yes"/>
 </segment>
 </net>
@@
 <wire x1="-58.42" y1="114.3" x2="-58.42" y2="124.46" width="0.1524" layer="91"/>
 <pinref part="R7" gate="G$1" pin="1"/>
-<pinref part="R6" gate="G$1" pin="1"/>
 <wire x1="-58.42" y1="124.46" x2="-58.42" y2="127" width="0.1524" layer="91"/>
 <wire x1="-53.34" y1="124.46" x2="-58.42" y2="124.46" width="0.1524" layer="91"/>
 <junction x="-58.42" y="124.46"/>
+<pinref part="R9" gate="G$1" pin="1"/>
 </segment>
 </net>
 <net name="AMP_CUR_SENSE" class="0">
 <segment>
-<pinref part="R6" gate="G$1" pin="2"/>
 <wire x1="-43.18" y1="124.46" x2="-38.1" y2="124.46" width="0.1524" layer="91"/>
 <wire x1="-38.1" y1="124.46" x2="-38.1" y2="111.76" width="0.1524" layer="91"/>
@@
 <junction x="-38.1" y="111.76"/>
 <label x="-35.56" y="111.76" size="1.27" layer="95" xref="yes"/>
+<pinref part="R9" gate="G$1" pin="2"/>
 </segment>
 <segment>
@@
 </segment>
 </net>
+<net name="N$6" class="0">
+<segment>
+<pinref part="U2" gate="U1" pin="ADC7"/>
+<wire x1="210.82" y1="124.46" x2="233.68" y2="124.46" width="0.1524" layer="91"/>
+<pinref part="JP2" gate="G$1" pin="1"/>
+<wire x1="233.68" y1="124.46" x2="233.68" y2="121.92" width="0.1524" layer="91"/>
+</segment>
+</net>

Commit message: Rev X02 finally done?
Parts:
- removed FRAME1: FRAME-LETTER, SparkFun-Aesthetics:FRAME-LETTER
- removed JP11, JP13: JUMPER-SMT_2_NC_TRACE_SILK, SparkFun-Jumpers:JUMPER-SMT_2_NC_TRACE_SILK
- removed JP2: ADR, SparkFun-Jumpers:JUMPER-SMT_2_NC_TRACE_SILK
- removed U$44: OPA344, SparkFun-IC-Amplifiers:OPA344
- added 3V3, SCK, STEP, VIN: JUMPER-SMT_2_NC_TRACE_SILK, SparkFun-Jumpers:JUMPER-SMT_2_NC_TRACE_SILK
- added ADR: ADR, SparkFun-Jumpers:JUMPER-SMT_2_NO_SILK
- added C12: 0.1uF, SparkFun-Capacitors:0.1UF-0603-25V-(+80/-20%)
- added FD1, FD2, FD3, FD4: FIDUCIAL1X2, SparkFun-Aesthetics:FIDUCIAL1X2
- added FRAME2: FRAME-LEDGER, SparkFun-Aesthetics:FRAME-LEDGER
- added R6, R8: 2.2k, SparkFun-Resistors:2.2KOHM-0603-1/10W-1%
- added U$49: SPARKX-LOGO4, SparkX:SPARKX-LOGO4
- added U44: OPA344, SparkFun-IC-Amplifiers:OPA344
- D2: value GREEN -> BLUE; device SparkFun-LED:LED-GREEN0603 -> SparkFun-LED:LED-BLUE0603
- D3: value BLUE -> GREEN; device SparkFun-LED:LED-BLUE0603 -> SparkFun-LED:LED-GREEN0603
- JP1: value JUMPER-SMT_2_NC_TRACE_SILK -> JUMPER-SMT_3_2-NC_TRACE_SILK; device SparkFun-Jumpers:JUMPER-SMT_2_NC_TRACE_SILK -> SparkFun-Jumpers:JUMPER-SMT_3_2-NC_TRACE_SILK
- R11: value 470 -> 1k; device SparkFun-Resistors:470OHM-0603-1/10W-1% -> SparkFun-Resistors:1KOHM-0603-1/10W-1%
- R12: value 4.7k -> 470; device SparkFun-Resistors:4.7KOHM-0603-1/10W-1% -> SparkFun-Resistors:470OHM-0603-1/10W-1%
Connections:
- new net N$15: JP1.3, R6.2
- new net N$16: JP1.1, R8.2
- new net N$17: R12.2, SCK.1
- net 3.3V: now also 3V3.2, C12.1, JP1.2, U44G2.P$V+; no longer JP13.2
- net AMP_CUR_SENSE: now also U44G1.OUT; no longer U$44G1.OUT
- net CURRENT_SENSE: now also U44G1.+IN; no longer U$44G1.+IN
- net GND: now also ADR.2, C12.2, U44G2.P$V-; no longer JP2.2
- net N$11: now also STEP.1; no longer JP11.1
- net N$12: now also R12.1; no longer R12.2
- net N$2: now also U44G1.-IN; no longer U$44G1.-IN
- net N$27: now also 3V3.1; no longer JP13.1
- net N$4: now also VIN.1; no longer JP1.1
- net N$6: now also ADR.1; no longer JP2.1
- net SCK: now also SCK.2; no longer R12.1
- net SCL: now also R8.1
- net SDA: now also R6.1
- net STEP: now also STEP.2; no longer JP11.2
- net VIN: now also VIN.2; no longer JP1.2
Other:
- note added: "7-Bit Unshifted I2C Address ADR open: 0x52 ADR closed: 0x51 Software configurable as well (ADR jumper open)"
- note added: "Cut jumper to disconnect the I2C pullup resistors."
- note added: "LEDs"
- note added: "NOTE: These jumpers normally closed. Cut them to disable LEDs."
- note added: "NOTE: This is only a "soft" E-stop. Will not power down all systems, but will stop the motor."
- note added: "Non-Inverting OpAmp (A = 23)"
- note added: "Programming Connectors"
- note added: "Serial"
- note added: "X02"
- note removed: "Power"
- note removed: "Programming"
- note removed: "Qwiic Connectors"
- moved on the sheet: C1, C10, C11, C14, C2, C3, C4, C5, C6, C7, C8, C9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
