File: Hardware/Qwiic-Step.brd (EAGLE design)
At the start: 50.8 x 50.8 mm, 101 parts, among them J1 PTH, J2 Qwiic Right Angle, J3 5.5x2.1mm Barrel, J4 Qwiic Right Angle, J5 ISP, U1 A4988ALT1, U2 ATMEGA328P_TQFP, U4 HV7801, Y1 16MHz

Commit message: Merge x02 hardware changes from harware changes branch
Parts:
- removed FRAME1: FRAME-LETTER, SparkFun-Aesthetics:CREATIVE_COMMONS
- removed JP11, JP13: JUMPER-SMT_2_NC_TRACE_SILK, SparkFun-Jumpers:SMT-JUMPER_2_NC_TRACE_SILK
- removed JP2: INT, SparkFun-Jumpers:SMT-JUMPER_2_NC_TRACE_SILK
- removed U$39: (no value), buzzard_labels (15):B#3
- removed U4: HV7801, SparkFun-IC-Special-Function:SOT23-5
- added 3V3, SCK, STEP, VIN: JUMPER-SMT_2_NC_TRACE_SILK, SparkFun-Jumpers:SMT-JUMPER_2_NC_TRACE_SILK
- added ADR: ADR, SparkFun-Jumpers:SMT-JUMPER_2_NO_SILK
- added C12: 0.1uF, SparkFun-Capacitors:0603
- added FD1, FD2, FD3, FD4: FIDUCIAL1X2, SparkFun-Aesthetics:FIDUCIAL-1X2
- added FRAME2: FRAME-LEDGER, SparkFun-Aesthetics:CREATIVE_COMMONS
- added R7: 1k, SparkFun-Resistors:0603
- added R8: 2.2k, SparkFun-Resistors:0603
- added R9: 22k, SparkFun-Resistors:0603
- added U$44: (no value), buzzard_labels (42):GND0
- added U$45: (no value), buzzard_labels (28):3V31
- added U$46: (no value), buzzard_labels (31):B#4
- added U$47: (no value), buzzard_labels (31):B#5
- added U$48: (no value), buzzard_labels (38):TXO2
- added U$49: SPARKX-LOGO4, SparkX:SPARKX-MEDIUM
- added U$53: (no value), buzzard_labels (42):PWR1
- added U$54: (no value), buzzard_labels (42):A#2
- added U$55: (no value), buzzard_labels (42):A#3
- added U$56: (no value), buzzard_labels (34):QWIIC_STEP0
- added U$57: (no value), buzzard_labels (42):B#4
- added U$58: (no value), buzzard_labels (42):B#5
- added U44: OPA344, SparkFun-IC-Amplifiers:SOT23-5
- D2: value GREEN -> BLUE
- D3: value BLUE -> GREEN
- JP1: value JUMPER-SMT_2_NC_TRACE_SILK -> (none); device SparkFun-Jumpers:SMT-JUMPER_2_NC_TRACE_SILK -> SparkFun-Jumpers:SMT-JUMPER_3_2-NC_TRACE_SILK
- R12: value 4.7k -> 470
- R6: value 0.25OHM_RES -> 2.2k; device qwiic_step:2512_RES -> SparkFun-Resistors:0603
- U$13: device buzzard_labels (16):VIN1 -> buzzard_labels (43):STAT0
- U$15: device buzzard_labels (15):A#0 -> Labels:I_SUPER2_C-()-03
- U$16: device buzzard_labels (15):A#1 -> Labels:I_SUPER2_C-()-03
- U$17: device buzzard_labels (15):B#2 -> buzzard_labels (38):3V31
- U$18: device buzzard_labels (15):B#3 -> buzzard_labels (38):DTR4
- U$19: device SparkX:SPARKX-MEDIUM -> buzzard_labels (39):DEBUG0
- U$21: device buzzard_labels:BLK2 -> buzzard_labels (38):GND0
- U$22: device buzzard_labels:GRN1 -> buzzard_labels (38):GND0
- U$32: device buzzard_labels (25):QWIIC_STEP0 -> buzzard_labels (31):A#2
- U$35: device buzzard_labels (26):PROG0 -> buzzard_labels (38):RXI3
- U$36: device buzzard_labels (15):A#0 -> buzzard_labels (31):A#3
- U$37: device buzzard_labels (15):A#1 -> buzzard_labels (28):STEP2
- U$38: device buzzard_labels (15):B#2 -> buzzard_labels (28):VIN0
- U$40: device buzzard_labels (27):SERIAL0 -> buzzard_labels (16):8#35V0
- moved U$40 39.6 mm to (44.5, 6.35), turned to 0 degrees
- moved JP1 38.9 mm to (33.0, 11.4), flipped to the bottom
- moved U$13 34.3 mm to (8.89, 33.0), turned to 0 degrees
- moved U$19 28.6 mm to (4.70, 6.48), flipped to the top, turned to 90 degrees
- moved U$17 27.9 mm to (6.22, 10.7), flipped to the bottom
- moved R6 25.6 mm to (31.8, 8.89)
- moved U$16 24.7 mm to (34.3, 13.3), flipped to the bottom
- moved U$18 23.7 mm to (6.35, 18.3), flipped to the bottom
- moved U$15 23.6 mm to (34.3, 13.3), flipped to the bottom
- moved U$25 22.6 mm to (20.2, 16.4), flipped to the bottom
- moved U$37 21.7 mm to (8.89, 30.5)
- moved U$7 16.1 mm to (0.25, 30.5)
- moved U$22 16.0 mm to (6.48, 5.59)
- moved U$11 14.9 mm to (50.9, 12.7), turned to 0 degrees
- moved C4 14.2 mm to (8.89, 19.1)
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Connections:
- removed net ADR: JP2.2, U2.23
- removed net CURR_SENSE: U2.19, U4.5
- removed net EP: U2.25
- removed net MOTOR_SUPPLY: R6.2, U1.22, U1.28, U4.1
- removed net N$31: R18.2, U1.27
- new net AMP_CUR_SENSE: R9.2, U2.19, U44.1
- new net CURRENT_SENSE: R18.2, U1.27, U44.3
- new net N$15: JP1.3, R6.2
- new net N$16: JP1.1, R8.2
- new net N$17: R12.2, SCK.1
- new net N$2: R7.1, R9.1, U44.4
- new net N$6: ADR.1, U2.22
- net 3.3V: now also 3V3.2, C12.1, JP1.2, U44.5; no longer JP13.2
- net A49885_!RESET!: now also U2.23; no longer U2.22
- net COILA+: now also J6.P$4; no longer J6.4
- net COILA-: now also J6.P$3; no longer J6.3
- net COILB+: now also J6.P$1; no longer J6.1
- net COILB-: now also J6.P$2; no longer J6.2
- net GND: now also ADR.2, C12.2, J9.P$2, R7.2, U44.2; no longer J9.2, JP2.1, U4.4
- net N$11: now also STEP.1; no longer JP11.1
- net N$12: now also R12.1; no longer R12.2
- net N$27: now also 3V3.1; no longer JP13.1
- net N$4: now also VIN.1; no longer JP1.1
- net N$7: now also J9.P$1; no longer J9.1
- net SCK: now also SCK.2; no longer R12.1
- net SCL: now also R8.1
- net SDA: now also R6.1
- net STEP: now also STEP.2; no longer JP11.2
- net VIN: now also U1.22, U1.28, VIN.2; no longer JP1.2, R6.1, U4.3
Routing:
- net STEP: track 40.8 -> 78.9 mm, vias 4 -> 5
- net !ENABLE!: track 14.5 -> 51.7 mm
- net MOTOR_SUPPLY: track 32.3 -> 0.00 mm, vias 5 -> 0
- net ADR: track 26.6 -> 0.00 mm, vias 2 -> 0
- net DIR: track 10.7 -> 34.6 mm, vias 2 -> 3
- net AMP_CUR_SENSE: track 0.00 -> 22.7 mm, vias 0 -> 2
- net VIN: track 80.6 -> 58.5 mm
- net 3.3V: track 152.7 -> 132.9 mm, vias 13 -> 10
- net CURR_SENSE: track 17.5 -> 0.00 mm
- net SDA: track 39.8 -> 56.0 mm
- net AREF: track 14.9 -> 5.39 mm
- net A49885_!RESET!: track 20.3 -> 29.5 mm
- net CURRENT_SENSE: track 0.00 -> 9.04 mm
- net !SLEEP!: track 27.9 -> 20.5 mm
- net N$31: track 5.96 -> 0.00 mm
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- added copper zone on layer 2, net 3.3V
- added copper zone on layer 1, net CURRENT_SENSE
- added copper zone on layer 15, net GND
- added copper zone on layer 1, net VIN
- added copper zone on layer 2, net VIN
- removed copper zone on layer 1, net MOTOR_SUPPLY
- removed copper zone on layer 1, net N$31

Commit message: Change resistor values on VIN and STEP LEDs.
Parts:
- R11: value 1k -> 0
Changed lines of the file:
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@@
 <?xml version="1.0" encoding="utf-8"?>
 <!DOCTYPE eagle SYSTEM "eagle.dtd">
-<eagle version="9.4.2">
+<eagle version="9.5.2">
 <drawing>
 <settings>
@@
 <element name="JP7" library="SparkFun-Hardware" package="STAND-OFF" value="STAND-OFF" x="48.26" y="2.54" smashed="yes"/>
 <element name="JP10" library="SparkFun-Hardware" package="STAND-OFF" value="STAND-OFF" x="48.26" y="48.26" smashed="yes"/>
-<element name="R11" library="SparkFun-Resistors" package="0603" value="1k" x="11.43" y="30.48" smashed="yes">
+<element name="R11" library="SparkFun-Resistors" package="0603" value="0" x="11.43" y="30.48" smashed="yes">
 <attribute name="NAME" x="11.43" y="31.242" size="0.6096" layer="25" font="vector" ratio="20" align="bottom-center"/>
-<attribute name="PROD_ID" value="RES-07856" x="11.43" y="30.48" size="1.778" layer="27" font="vector" ratio="15" display="off"/>
-<attribute name="VALUE" value="1k" x="11.43" y="29.718" size="0.6096" layer="27" font="vector" ratio="20" align="top-center"/>
+<attribute name="PROD_ID" value="RES-08609" x="11.43" y="30.48" size="1.778" layer="27" font="vector" ratio="15" display="off"/>
+<attribute name="VALUE" value="0" x="11.43" y="29.718" size="0.6096" layer="27" font="vector" ratio="20" align="top-center"/>
 </element>
 <element name="D3" library="SparkFun-LED" package="LED-0603" value="GREEN" x="7.62" y="30.48" smashed="yes" rot="R180">

Commit message: Increasing yellow LED resistor to 10k to limit brightness
Parts:
- R1: value 4.7k -> 10k
Changed lines of the file:
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@@
 <attribute name="VALUE" x="36.449" y="1.778" size="0.6096" layer="27" font="vector" ratio="20"/>
 </element>
-<element name="R1" library="SparkFun-Resistors" package="0603" value="4.7k" x="11.43" y="38.1" smashed="yes">
+<element name="R1" library="SparkFun-Resistors" package="0603" value="10k" x="11.43" y="38.1" smashed="yes">
 <attribute name="NAME" x="11.43" y="38.862" size="0.6096" layer="25" font="vector" ratio="20" align="bottom-center"/>
-<attribute name="PROD_ID" value="RES-07857" x="12.7" y="38.1" size="1.778" layer="27" font="vector" ratio="15" display="off"/>
-<attribute name="VALUE" value="4.7k" x="11.43" y="37.338" size="0.6096" layer="27" font="vector" ratio="20" align="top-center"/>
+<attribute name="PROD_ID" value="RES-00824" x="12.7" y="38.1" size="1.778" layer="27" font="vector" ratio="15" display="off"/>
+<attribute name="VALUE" value="10k" x="11.43" y="37.338" size="0.6096" layer="27" font="vector" ratio="20" align="top-center"/>
 </element>
 <element name="VIN" library="SparkFun-Jumpers" package="SMT-JUMPER_2_NC_TRACE_SILK" package3d_urn="urn:adsk.eagle:package:39281/1" value="JUMPER-SMT_2_NC_TRACE_SILK" x="11.43" y="38.1" smashed="yes" rot="MR0">

Commit message: Change CUR_REF_PWM RC filter to 100k/1uF.
Parts:
- C2: value 10nF -> 1.0uF
- R3: value 33k -> 100k
Changed lines of the file:
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@@
 <attribute name="VALUE" value="BLUE" x="7.62" y="33.655" size="0.6096" layer="27" font="vector" ratio="20" rot="R180" align="top-center"/>
 </element>
-<element name="R3" library="SparkFun-Resistors" package="0603" value="33k" x="34.925" y="26.67" smashed="yes" rot="R90">
+<element name="R3" library="SparkFun-Resistors" package="0603" value="100k" x="34.925" y="26.67" smashed="yes" rot="R90">
 <attribute name="NAME" x="34.163" y="26.67" size="0.6096" layer="25" font="vector" ratio="20" rot="R90" align="bottom-center"/>
-<attribute name="PROD_ID" value="RES-08416" x="34.925" y="26.67" size="1.778" layer="27" font="vector" ratio="15" rot="R90" display="off"/>
-<attribute name="VALUE" x="35.687" y="26.67" size="0.6096" layer="27" font="vector" ratio="20" rot="R90" align="top-center"/>
+<attribute name="PROD_ID" value="RES-07828" x="34.925" y="26.67" size="1.778" layer="27" font="vector" ratio="15" rot="R90" display="off"/>
+<attribute name="VALUE" value="100k" x="35.687" y="26.67" size="0.6096" layer="27" font="vector" ratio="20" rot="R90" align="top-center"/>
 </element>
-<element name="C2" library="SparkFun-Capacitors" package="0603" value="10nF" x="36.83" y="26.67" smashed="yes" rot="R270">
+<element name="C2" library="SparkFun-Capacitors" package="0603" value="1.0uF" x="36.83" y="26.67" smashed="yes" rot="R270">
 <attribute name="NAME" x="37.592" y="26.67" size="0.6096" layer="25" font="vector" ratio="20" rot="R270" align="bottom-center"/>
-<attribute name="PROD_ID" value="CAP-00867" x="36.83" y="26.67" size="1.778" layer="27" font="vector" ratio="15" rot="R270" display="off"/>
-<attribute name="VALUE" x="36.068" y="26.67" size="0.6096" layer="27" font="vector" ratio="20" rot="R270" align="top-center"/>
+<attribute name="PROD_ID" value="CAP-00868" x="36.83" y="26.67" size="1.778" layer="27" font="vector" ratio="15" rot="R270" display="off"/>
+<attribute name="VALUE" value="1.0uF" x="36.068" y="26.67" size="0.6096" layer="27" font="vector" ratio="20" rot="R270" align="top-center"/>
 </element>
 <element name="ADR" library="SparkFun-Jumpers" package="SMT-JUMPER_2_NO_SILK" package3d_urn="urn:adsk.eagle:package:39279/1" value="ADR" x="17.78" y="13.97" smashed="yes" rot="MR0">
