File: Hardware/Production/Qwiic-Step-Panel.brd (EAGLE design)
At the start: 50.8 x 50.8 mm, 101 parts, among them J1 PTH, J2 Qwiic Right Angle, J3 5.5x2.1mm Barrel, J4 Qwiic Right Angle, J5 ISP, U1 A4988ALT1, U2 ATMEGA328P_TQFP, U4 HV7801, Y1 16MHz

Commit message: Final board layout
Parts:
- removed FRAME1: FRAME-LETTER, SparkFun-Aesthetics:CREATIVE_COMMONS
- added C12, C13, C15, C16, C17, C19, C21, C22, C24, C25, C26, C27, C28, C29, C31, C33, C34, C36, C37, C38, C39, C40, C41, C43, C45, C46, C48: 0.1uF, SparkFun-Capacitors:0603
- added C18, C30, C42: 0.22uF, SparkFun-Capacitors:0603
- added C20, C32, C44: 47uF, SparkFun-Capacitors:PANASONIC_D
- added C23, C35, C47: 10nF, SparkFun-Capacitors:0603
- added D10, D15, D20: Yellow, SparkFun-LED:LED-0603
- added D11, D16, D6: 3A/40V/500mV, SparkFun-DiscreteSemi:SMA-DIODE
- added D12, D17, D7: BLUE, SparkFun-LED:LED-0603
- added D13, D18, D8: RED, SparkFun-LED:LED-0603
- added D14, D19, D9: GREEN, SparkFun-LED:LED-0603
- added E$1, E$2: (no value), SparkFun-Aesthetics:FIDUCIAL-1X2
- added E$3: (no value), SparkFun-Retired:FIDUCIAL-1.5X3
- added J12, J23, J34: 5.5x2.1mm Barrel, SparkFun-Connectors:POWER_JACK_SMD
- added J13, J24, J35: PTH, SparkX:1X04_NO_SILK
- added J14, J15, J25, J26, J36, J37: Qwiic Right Angle, SparkFun-Connectors:JST04_1MM_RA
- added J16, J27, J38: ISP, SparkFun-Connectors:2X3_TEST_POINTS
- added J17, J28, J39: (no value), SparkFun-Connectors:1X06_NO_SILK
- added J18, J19, J29, J30, J40, J41: (no value), SparkFun-Connectors:JST-2-SMD
- added J20, J31, J42: (no value), SparkFun-Connectors:1X01_NO_SILK
- added J21, J32, J43: (no value), SparkFun-Connectors:LATCHTERMINAL-5MM-2
- added J22, J33, J44: (no value), SparkFun-Connectors:LATCHTERMINAL-5MM-4
- added JP12, JP18, JP22, JP27, JP31, JP36: INT, SparkFun-Jumpers:SMT-JUMPER_2_NC_TRACE_SILK
- added JP14, JP15, JP19, JP20, JP23, JP24, JP28, JP29, JP3, JP32, JP33, JP4: STAND-OFF, SparkFun-Hardware:STAND-OFF
- added JP16, JP17, JP21, JP25, JP26, JP30, JP34, JP35, JP5: JUMPER-SMT_2_NC_TRACE_SILK, SparkFun-Jumpers:SMT-JUMPER_2_NC_TRACE_SILK
- added LOGO2, LOGO3, LOGO4: OSHW-LOGOMINI, SparkFun-Aesthetics:OSHW-LOGO-MINI
- added R13, R16, R17, R31, R32, R33, R34, R45, R46, R47, R48, R9: 20k, SparkFun-Resistors:0603
- added R21, R24, R35, R38, R49, R52: 4.7k, SparkFun-Resistors:0603
- added R22, R25, R36, R39, R50, R53: 10k, SparkFun-Resistors:0603
- added R23, R26, R37, R40, R51, R54: 1k, SparkFun-Resistors:0603
- added R27, R41, R55: 33k, SparkFun-Resistors:0603
- added R28, R42, R56: 0.25OHM_RES, qwiic_step:2512_RES
- added R29, R30, R43, R44, R7, R8: 0.11, SparkFun-Resistors:2010
- added S2, S3, S4: Tall Switch, SparkFun-Switches:TACTILE_SWITCH_SMD_5.2MM
- added U$100, U$101, U$143, U$144, U$57, U$58: (no value), buzzard_labels:BLK2
- added U$102, U$103, U$145, U$146, U$59, U$60: (no value), buzzard_labels:GRN1
- added U$104, U$114, U$147, U$157, U$61, U$71: (no value), SparkFun-Aesthetics:QWIIC_5.5MM
- added U$105, U$106, U$148, U$149, U$62, U$63: (no value), buzzard_labels (16):8#35V0
- added U$107, U$108, U$150, U$151, U$64, U$65: (no value), buzzard_labels (16):VIN1
- added U$109, U$152, U$66: (no value), buzzard_labels (16):E#STOP2
- added U$110, U$153, U$67: (no value), buzzard_labels (16):LIM_SW3
- added U$111, U$115, U$154, U$158, U$68, U$72: (no value), buzzard_labels (16):INT4
- added U$112, U$155, U$69: (no value), buzzard_labels (18):ADR0
- added U$113, U$156, U$70: (no value), buzzard_labels (18):RESET1
- added U$116, U$159, U$73: (no value), buzzard_labels (25):QWIIC_STEP0
- added U$117, U$160, U$74: (no value), buzzard_labels (19):3V35
- added U$118, U$161, U$75: (no value), buzzard_labels (19):GND6
- added U$119, U$162, U$76: (no value), buzzard_labels (19):SDA4
- added U$120, U$163, U$77: (no value), buzzard_labels (19):SCL3
- added U$121, U$164, U$78: (no value), buzzard_labels (26):PROG0
- added U$122, U$138, U$165, U$52, U$79, U$95: (no value), buzzard_labels (15):A#0
- added U$123, U$139, U$166, U$53, U$80, U$96: (no value), buzzard_labels (15):A#1
- added U$124, U$140, U$167, U$54, U$81, U$97: (no value), buzzard_labels (15):B#2
- added U$125, U$141, U$168, U$55, U$82, U$98: (no value), buzzard_labels (15):B#3
- added U$126, U$169, U$83: (no value), buzzard_labels (27):SERIAL0
- added U$127, U$170, U$84: (no value), buzzard_labels (19):INT2
- added U$128, U$171, U$85: (no value), buzzard_labels (19):GND1
- added U$129, U$172, U$86: (no value), buzzard_labels (19):PWR0
- added U$130, U$44, U$87: (no value), buzzard_labels (8):3V30
- added U$131, U$45, U$88: (no value), buzzard_labels (8):3V37
- added U$132, U$46, U$89: (no value), buzzard_labels (8):GND8
- added U$133, U$47, U$90: (no value), buzzard_labels (8):SCL5
- added U$134, U$48, U$91: (no value), buzzard_labels (8):SDA6
- added U$135, U$49, U$92: (no value), buzzard_labels (8):STEP4
- added U$136, U$50, U$93: (no value), buzzard_labels (8):VIN3
- added U$137, U$51, U$94: (no value), buzzard_labels (13):STAT5
- added U$142, U$56, U$99: (no value), SparkX:SPARKX-MEDIUM
- added U10, U3, U7: A4988ALT1, SparkFun-IC-Special-Function:QFN-28-5MM
- added U11, U5, U8: ATMEGA328P_TQFP, SparkFun-IC-Microcontroller:TQFP32-08
- added U12, U6, U9: HV7801, SparkFun-IC-Special-Function:SOT23-5
- added Y2, Y3, Y4: 16MHz, SparkFun-Clocks:RESONATOR-SMD-3.2X1.3
Connections:
- new net !ENABLE!1: J16.4, R17.1, U3.2, U5.14
- new net !ENABLE!2: J27.4, R34.1, U7.2, U8.14
- new net !ENABLE!3: J38.4, R48.1, U10.2, U11.14
- new net !RST!1: C24.2, J16.5, R25.1, S2.3, S2.4, U5.29
- new net !RST!2: C36.2, J27.5, R39.1, S3.3, S3.4, U8.29
- new net !RST!3: C48.2, J38.5, R53.1, S4.3, S4.4, U11.29
- new net !SLEEP!1: R13.1, U3.14, U5.2
- new net !SLEEP!2: R32.1, U7.14, U8.2
- new net !SLEEP!3: R46.1, U10.14, U11.2
- new net 3.3V1: C15.1, C22.1, J13.2, J14.2, J15.2, J16.2, J17.4, JP12.2, JP17.2, R13.2, R16.2, R17.2, R25.2, U3.15, U5.18, U5.4, U5.6
- new net 3.3V2: C27.1, C34.1, J24.2, J25.2, J26.2, J27.2, J28.4, JP22.2, JP26.2, R32.2, R33.2, R34.2, R39.2, U7.15, U8.18, U8.4, U8.6
- new net 3.3V3: C39.1, C46.1, J35.2, J36.2, J37.2, J38.2, J39.4, JP31.2, JP35.2, R46.2, R47.2, R48.2, R53.2, U10.15, U11.18, U11.4, U11.6
- new net A49885_!RESET!1: R16.1, U3.12, U5.22
- new net A49885_!RESET!2: R33.1, U7.12, U8.22
- new net A49885_!RESET!3: R47.1, U10.12, U11.22
- new net ADR1: JP18.2, U5.15
- new net ADR2: JP27.2, U8.15
- new net ADR3: JP36.2, U11.15
- new net AREF1: C21.1, U5.20
- new net AREF2: C33.1, U8.20
- new net AREF3: C45.1, U11.20
- new net COILA+1: J22.4, U3.21
- new net COILA+2: J33.4, U7.21
- new net COILA+3: J44.4, U10.21
- new net COILA-1: J22.3, U3.24
- new net COILA-2: J33.3, U7.24
- new net COILA-3: J44.3, U10.24
- new net COILB+1: J22.1, U3.1
- new net COILB+2: J33.1, U7.1
- new net COILB+3: J44.1, U10.1
- new net COILB-1: J22.2, U3.26
- new net COILB-2: J33.2, U7.26
- new net COILB-3: J44.2, U10.26
- new net CURR_SENSE1: U5.19, U6.5
- new net CURR_SENSE2: U8.19, U9.5
- new net CURR_SENSE3: U11.19, U12.5
- new net CUR_REF1: C23.1, R27.2, U3.17
- new net CUR_REF2: C35.1, R41.2, U7.17
- new net CUR_REF3: C47.1, R55.2, U10.17
- new net CUR_REF_PWM1: R27.1, U5.9
- new net CUR_REF_PWM2: R41.1, U8.9
- new net CUR_REF_PWM3: R55.1, U11.9
- new net DIR1: U3.19, U5.10
- new net DIR2: U7.19, U8.10
- new net DIR3: U10.19, U11.10
- new net DTR1: C24.1, J17.1
- new net DTR2: C36.1, J28.1
- new net DTR3: C48.1, J39.1
- new net EP1: U5.25
- new net EP2: U8.25
- new net EP3: U11.25
- new net GND1: C12.2, C15.2, C16.2, C17.2, C18.2, C20.-, C21.2, C22.2, C23.2, D10.C, D7.C, D8.C, D9.C, J12.GND, J12.P$4, J13.1, J14.1, J15.1, J16.6, J17.5, J17.6, J18.2, J19.2, J21.2, JP18.1, R7.1, R8.1, R9.2, S2.1, S2.2, U3.18, U3.29, U3.3, U5.21, U5.3, U5.5, U6.4, Y2.2
- new net GND2: C25.2, C27.2, C28.2, C29.2, C30.2, C32.-, C33.2, C34.2, C35.2, D12.C, D13.C, D14.C, D15.C, J23.GND, J23.P$4, J24.1, J25.1, J26.1, J27.6, J28.5, J28.6, J29.2, J30.2, J32.2, JP27.1, R29.1, R30.1, R31.2, S3.1, S3.2, U7.18, U7.29, U7.3, U8.21, U8.3, U8.5, U9.4, Y3.2
- new net GND3: C37.2, C39.2, C40.2, C41.2, C42.2, C44.-, C45.2, C46.2, C47.2, D17.C, D18.C, D19.C, D20.C, J34.GND, J34.P$4, J35.1, J36.1, J37.1, J38.6, J39.5, J39.6, J40.2, J41.2, J43.2, JP36.1, R43.1, R44.1, R45.2, S4.1, S4.2, U10.18, U10.29, U10.3, U11.21, U11.3, U11.5, U12.4, Y4.2
- new net INT10: J41.1, U11.1
- new net INT2: J20.1, R22.1, U5.24
- new net INT3: J18.1, U5.32
- new net INT4: J19.1, U5.1
- new net INT5: J31.1, R36.1, U8.24
- new net INT6: J29.1, U8.32
- new net INT7: J30.1, U8.1
- new net INT8: J42.1, R50.1, U11.24
- new net INT9: J40.1, U11.32
- new net MISO1: J16.1, U5.16
- new net MISO2: J27.1, U8.16
- new net MISO3: J38.1, U11.16
- new net MOTOR_SUPPLY1: R28.2, U3.22, U3.28, U6.1
- new net MOTOR_SUPPLY2: R42.2, U7.22, U7.28, U9.1
- new net MOTOR_SUPPLY3: R56.2, U10.22, U10.28, U12.1
- new net MS10: U10.10, U11.12
- new net MS11: U10.11, U11.11
- new net MS12: U10.9, U11.13
- new net MS4: U3.10, U5.12
- new net MS5: U3.11, U5.11
- new net MS6: U3.9, U5.13
- new net MS7: U7.10, U8.12
- new net MS8: U7.11, U8.11
- new net MS9: U7.9, U8.13
- new net N$15: C13.2, U3.5
- new net N$16: R9.1, U3.13
- new net N$17: C18.1, U3.8
- new net N$18: C19.1, U3.6
- new net N$2: R7.2, U3.27
- new net N$22: D10.A, R21.1
- new net N$23: JP5.1, R21.2
- new net N$24: D6.A, J12.VIN0, J21.1
- new net N$25: D7.A, R23.1
- new net N$28: JP16.1, R23.2
- new net N$29: D9.A, R24.2
- new net N$3: R8.2, U3.23
- new net N$30: U5.7, Y2.1
- new net N$33: U5.8, Y2.3
- new net N$34: D8.A, R26.1
- new net N$35: JP17.1, R26.2
- new net N$36: JP12.1, R22.2
- new net N$37: R29.2, U7.27
- new net N$38: R30.2, U7.23
- new net N$39: C26.1, U7.4
- new net N$40: C26.2, U7.5
- new net N$41: R31.1, U7.13
- new net N$42: C30.1, U7.8
- new net N$43: C31.1, U7.6
- new net N$44: D15.A, R35.1
- new net N$45: JP21.1, R35.2
- new net N$46: D11.A, J23.VIN0, J32.1
- new net N$47: D12.A, R37.1
- new net N$48: JP25.1, R37.2
- new net N$49: D14.A, R38.2
- new net N$50: U8.7, Y3.1
- new net N$51: U8.8, Y3.3
- new net N$52: D13.A, R40.1
- new net N$53: JP26.1, R40.2
- new net N$54: JP22.1, R36.2
- new net N$55: R43.2, U10.27
- new net N$56: R44.2, U10.23
- new net N$57: C38.1, U10.4
- new net N$58: C38.2, U10.5
- new net N$59: R45.1, U10.13
- new net N$6: C13.1, U3.4
- new net N$60: C42.1, U10.8
- new net N$61: C43.1, U10.6
- new net N$62: D20.A, R49.1
- new net N$63: JP30.1, R49.2
- new net N$64: D16.A, J34.VIN0, J43.1
- new net N$65: D17.A, R51.1
- new net N$66: JP34.1, R51.2
- new net N$67: D19.A, R52.2
- new net N$68: U11.7, Y4.1
- new net N$69: U11.8, Y4.3
- new net N$70: D18.A, R54.1
- new net N$71: JP35.1, R54.2
- new net N$72: JP31.1, R50.2
- new net RXI1: J17.3, U5.30
- new net RXI2: J28.3, U8.30
- new net RXI3: J39.3, U11.30
- new net SCK1: J16.3, R24.1, U5.17
- new net SCK2: J27.3, R38.1, U8.17
- new net SCK3: J38.3, R52.1, U11.17
- new net SCL1: J13.4, J14.4, J15.4, U5.28
- new net SCL2: J24.4, J25.4, J26.4, U8.28
- new net SCL3: J35.4, J36.4, J37.4, U11.28
- new net SDA1: J13.3, J14.3, J15.3, U5.27
- new net SDA2: J24.3, J25.3, J26.3, U8.27
- new net SDA3: J35.3, J36.3, J37.3, U11.27
- new net STEP1: JP16.2, U3.16, U5.26
- new net STEP2: JP25.2, U7.16, U8.26
- new net STEP3: JP34.2, U10.16, U11.26
- new net TXO1: J17.2, U5.31
- new net TXO2: J28.2, U8.31
- new net TXO3: J39.2, U11.31
- new net VIN1: C12.1, C16.1, C17.1, C19.2, C20.+, D6.C, JP5.2, R28.1, U6.3
- new net VIN2: C25.1, C28.1, C29.1, C31.2, C32.+, D11.C, JP21.2, R42.1, U9.3
- new net VIN3: C37.1, C40.1, C41.1, C43.2, C44.+, D16.C, JP30.2, R56.1, U12.3
Routing:
- net 3.3V3: track 0.00 -> 152.4 mm, vias 0 -> 13
- net 3.3V2: track 0.00 -> 152.4 mm, vias 0 -> 13
- net 3.3V1: track 0.00 -> 152.4 mm, vias 0 -> 13
- net VIN3: track 0.00 -> 80.6 mm, vias 0 -> 6
- net VIN1: track 0.00 -> 80.6 mm, vias 0 -> 6
- net VIN2: track 0.00 -> 80.6 mm, vias 0 -> 6
- net INT9: track 0.00 -> 62.3 mm, vias 0 -> 2
- net INT3: track 0.00 -> 62.3 mm, vias 0 -> 2
- net INT6: track 0.00 -> 62.3 mm, vias 0 -> 2
- net STEP3: track 0.00 -> 40.7 mm, vias 0 -> 4
- net STEP2: track 0.00 -> 40.7 mm, vias 0 -> 4
- net STEP1: track 0.00 -> 40.7 mm, vias 0 -> 4
- net INT7: track 0.00 -> 40.4 mm, vias 0 -> 2
- net INT10: track 0.00 -> 40.4 mm, vias 0 -> 2
- net INT4: track 0.00 -> 40.4 mm, vias 0 -> 2
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- added copper zone on layer 1, net COILA+1
- added copper zone on layer 16, net COILA+1
- added copper zone on layer 1, net COILA+2
- added copper zone on layer 16, net COILA+2
- added copper zone on layer 1, net COILA+3
- added copper zone on layer 16, net COILA+3
- added copper zone on layer 1, net COILA-1
- added copper zone on layer 1, net COILA-2
- added copper zone on layer 1, net COILA-3
- added copper zone on layer 1, net COILB+1
- added copper zone on layer 16, net COILB+1
- added copper zone on layer 1, net COILB+2
- added copper zone on layer 16, net COILB+2
- added copper zone on layer 1, net COILB+3
- added copper zone on layer 16, net COILB+3
- added copper zone on layer 1, net COILB-1
- added copper zone on layer 1, net COILB-2
- added copper zone on layer 1, net COILB-3
- added copper zone on layer 1, net GND1
- added copper zone on layer 16, net GND1
- added copper zone on layer 1, net GND2
- added copper zone on layer 16, net GND2
- added copper zone on layer 1, net GND3
- added copper zone on layer 16, net GND3
- added copper zone on layer 1, net MOTOR_SUPPLY1
- added copper zone on layer 1, net MOTOR_SUPPLY2
- added copper zone on layer 1, net MOTOR_SUPPLY3
- added copper zone on layer 1, net N$2
- added copper zone on layer 1, net N$3
- added copper zone on layer 1, net N$37
- added copper zone on layer 1, net N$38
- added copper zone on layer 1, net N$55
- added copper zone on layer 1, net N$56
Other:
- board size 50.8 x 50.8 mm -> 129.8 x 115.8 mm
- board text added: "Route Out"
- board text added: "v-score"
- board text removed: "Brian Schmalz: http://schmalzhaus.com/BigEasyDriver/index.html"

Commit message: Rev X02 finalized and ordered
Parts:
- removed JP25, JP26, JP30, JP34, JP35: JUMPER-SMT_2_NC_TRACE_SILK, SparkFun-Jumpers:SMT-JUMPER_2_NC_TRACE_SILK
- removed JP27, JP31, JP36: INT, SparkFun-Jumpers:SMT-JUMPER_2_NC_TRACE_SILK
- removed JP28, JP29, JP32, JP33: STAND-OFF, SparkFun-Hardware:STAND-OFF
- removed U12: HV7801, SparkFun-IC-Special-Function:SOT23-5
- added 3V1, 3V2, 3V3, 3V4, SCK, SCK1, SCK2, SCK3, STEP, STEP1, STEP2, STEP3, VIN, VIN1, VIN2, VIN3: JUMPER-SMT_2_NC_TRACE_SILK, SparkFun-Jumpers:SMT-JUMPER_2_NC_TRACE_SILK
- added ADR, ADR1, ADR2, ADR3: ADR, SparkFun-Jumpers:SMT-JUMPER_2_NO_SILK
- added C49, C51, C52: 0.1uF, SparkFun-Capacitors:0603
- added C50: 10nF, SparkFun-Capacitors:0603
- added FD1, FD10, FD11, FD12, FD13, FD14, FD15, FD16, FD2, FD3, FD4, FD5, FD6, FD7, FD8, FD9: FIDUCIAL1X2, SparkFun-Aesthetics:FIDUCIAL-1X2
- added R57: 20k, SparkFun-Resistors:0603
- added R58: 4.7k, SparkFun-Resistors:0603
- added R59, R62: 10k, SparkFun-Resistors:0603
- added R60, R63, R65: 1k, SparkFun-Resistors:0603
- added R61: 470, SparkFun-Resistors:0603
- added R64: 33k, SparkFun-Resistors:0603
- added R66: 22k, SparkFun-Resistors:0603
- added R67, R68: 2.2k, SparkFun-Resistors:0603
- added U$173, U$182: (no value), SparkFun-Aesthetics:QWIIC_5.5MM
- added U$174, U$175, U$207: (no value), buzzard_labels (16):8#35V0
- added U$176: (no value), buzzard_labels (16):VIN1
- added U$177: (no value), buzzard_labels (16):E#STOP2
- added U$178: (no value), buzzard_labels (16):LIM_SW3
- added U$179, U$183: (no value), buzzard_labels (16):INT4
- added U$180: (no value), buzzard_labels (18):ADR0
- added U$181: (no value), buzzard_labels (18):RESET1
- added U$184: (no value), buzzard_labels (19):3V35
- added U$185: (no value), buzzard_labels (19):GND6
- added U$186: (no value), buzzard_labels (19):SDA4
- added U$187: (no value), buzzard_labels (19):SCL3
- added U$188: (no value), buzzard_labels (19):INT2
- added U$189: (no value), buzzard_labels (19):GND1
- added U$190: (no value), buzzard_labels (19):PWR0
- added U$191: (no value), buzzard_labels (28):3V31
- added U$192: (no value), buzzard_labels (28):STEP2
- added U$193: (no value), buzzard_labels (28):VIN0
- added U$194: (no value), buzzard_labels (34):QWIIC_STEP0
- added U$195: (no value), buzzard_labels (31):A#2
- added U$196: (no value), buzzard_labels (31):A#3
- added U$197: (no value), buzzard_labels (31):B#4
- added U$198: (no value), buzzard_labels (31):B#5
- added U$199: (no value), buzzard_labels (38):3V31
- added U$200: (no value), buzzard_labels (38):DTR4
- added U$201, U$202: (no value), buzzard_labels (38):GND0
- added U$203: (no value), buzzard_labels (38):RXI3
- added U$204: (no value), buzzard_labels (38):TXO2
- added U$205: SPARKX-LOGO4, SparkX:SPARKX-MEDIUM
- added U$206: (no value), buzzard_labels (39):DEBUG0
- added U$208: (no value), buzzard_labels (42):GND0
- added U$209: (no value), buzzard_labels (42):PWR1
- added U$210: (no value), buzzard_labels (42):A#2
- added U$211: (no value), buzzard_labels (42):A#3
- added U$212: (no value), buzzard_labels (42):B#4
- added U$213: (no value), buzzard_labels (42):B#5
- added U$214: (no value), buzzard_labels (43):STAT0
- added U$215, U$216: (no value), Labels:I_SUPER2_C-()-03
- added U44: OPA344, SparkFun-IC-Amplifiers:SOT23-5
- C18, C30, C42: value 0.22uF -> 0.1uF
- C19, C45: value 0.1uF -> 0.22uF
- C20, C44: value 47uF -> 0.1uF; device SparkFun-Capacitors:PANASONIC_D -> SparkFun-Capacitors:0603
- C21, C34: value 0.1uF -> 47uF; device SparkFun-Capacitors:0603 -> SparkFun-Capacitors:PANASONIC_D
- C23, C35: value 10nF -> 0.1uF
- C24, C37: value 0.1uF -> 10nF
- C32: value 47uF -> 0.22uF; device SparkFun-Capacitors:PANASONIC_D -> SparkFun-Capacitors:0603
- C47: value 10nF -> 47uF; device SparkFun-Capacitors:0603 -> SparkFun-Capacitors:PANASONIC_D
- D12, D17, D3, D7: value BLUE -> GREEN
- D14, D19, D2, D9: value GREEN -> BLUE
- JP1: value JUMPER-SMT_2_NC_TRACE_SILK -> (none); device SparkFun-Jumpers:SMT-JUMPER_2_NC_TRACE_SILK -> SparkFun-Jumpers:SMT-JUMPER_3_2-NC_TRACE_SILK
- JP11, JP13, JP16, JP17, JP5: value JUMPER-SMT_2_NC_TRACE_SILK -> STAND-OFF; device SparkFun-Jumpers:SMT-JUMPER_2_NC_TRACE_SILK -> SparkFun-Hardware:STAND-OFF
- JP12, JP18: value INT -> (none); device SparkFun-Jumpers:SMT-JUMPER_2_NC_TRACE_SILK -> SparkFun-Jumpers:SMT-JUMPER_3_2-NC_TRACE_SILK
- JP15, JP4: value STAND-OFF -> INT; device SparkFun-Hardware:STAND-OFF -> SparkFun-Jumpers:SMT-JUMPER_2_NC_TRACE_SILK
- JP2, JP22: value INT -> STAND-OFF; device SparkFun-Jumpers:SMT-JUMPER_2_NC_TRACE_SILK -> SparkFun-Hardware:STAND-OFF
- JP21: value JUMPER-SMT_2_NC_TRACE_SILK -> INT
- JP24: value STAND-OFF -> (none); device SparkFun-Hardware:STAND-OFF -> SparkFun-Jumpers:SMT-JUMPER_3_2-NC_TRACE_SILK
- R12: value 4.7k -> 470
- R13, R16: value 20k -> 0.11; device SparkFun-Resistors:0603 -> SparkFun-Resistors:2010
- R21, R38: value 4.7k -> 20k
- R22, R39: value 10k -> 20k
- R23, R37, R40, R54: value 1k -> 20k
- R27: value 33k -> 470
- R28, R42: value 0.25OHM_RES -> 10k; device qwiic_step:2512_RES -> SparkFun-Resistors:0603
- R29, R43, R7: value 0.11 -> 1k; device SparkFun-Resistors:2010 -> SparkFun-Resistors:0603
- R30: value 0.11 -> 33k; device SparkFun-Resistors:2010 -> SparkFun-Resistors:0603
- R31, R46, R48: value 20k -> 1k
- R32, R9: value 20k -> 22k
- R33, R34: value 20k -> 2.2k
- R35, R52: value 4.7k -> 0.11; device SparkFun-Resistors:0603 -> SparkFun-Resistors:2010
- R36, R53: value 10k -> 0.11; device SparkFun-Resistors:0603 -> SparkFun-Resistors:2010
- R41: value 33k -> 4.7k
- R44: value 0.11 -> 470; device SparkFun-Resistors:2010 -> SparkFun-Resistors:0603
- R45: value 20k -> 10k
- R47: value 20k -> 33k
- R49: value 4.7k -> 22k
- R50: value 10k -> 2.2k
- R51: value 1k -> 2.2k
- R55: value 33k -> 20k
- R56: value 0.25OHM_RES -> 20k; device qwiic_step:2512_RES -> SparkFun-Resistors:0603
- R6: value 0.25OHM_RES -> 2.2k; device qwiic_step:2512_RES -> SparkFun-Resistors:0603
- R8: value 0.11 -> 2.2k; device SparkFun-Resistors:2010 -> SparkFun-Resistors:0603
- U$100: device buzzard_labels:BLK2 -> buzzard_labels (42):GND0
- U$101: device buzzard_labels:BLK2 -> buzzard_labels (42):PWR1
- U$102: device buzzard_labels:GRN1 -> buzzard_labels (42):A#2
- U$103: device buzzard_labels:GRN1 -> buzzard_labels (42):A#3
- U$104: device SparkFun-Aesthetics:QWIIC_5.5MM -> buzzard_labels (42):B#4
- U$105: device buzzard_labels (16):8#35V0 -> buzzard_labels (42):B#5
- U$106: device buzzard_labels (16):8#35V0 -> buzzard_labels (43):STAT0
- U$107, U$108: device buzzard_labels (16):VIN1 -> Labels:I_SUPER2_C-()-03
- U$109: device buzzard_labels (16):E#STOP2 -> buzzard_labels (8):3V30
- U$110: device buzzard_labels (16):LIM_SW3 -> buzzard_labels (8):3V37
- U$111: device buzzard_labels (16):INT4 -> buzzard_labels (8):GND8
- U$112: device buzzard_labels (18):ADR0 -> buzzard_labels (8):SCL5
- U$113: device buzzard_labels (18):RESET1 -> buzzard_labels (8):SDA6
- U$114: device SparkFun-Aesthetics:QWIIC_5.5MM -> buzzard_labels (8):STEP4
- U$115: device buzzard_labels (16):INT4 -> buzzard_labels (8):VIN3
- U$116: device buzzard_labels (25):QWIIC_STEP0 -> buzzard_labels (13):STAT5
- U$117: device buzzard_labels (19):3V35 -> buzzard_labels:BLK2
- U$118: device buzzard_labels (19):GND6 -> buzzard_labels:GRN1
- U$119: device buzzard_labels (19):SDA4 -> SparkFun-Aesthetics:QWIIC_5.5MM
- U$120: device buzzard_labels (19):SCL3 -> buzzard_labels (16):8#35V0
- U$121: device buzzard_labels (26):PROG0 -> buzzard_labels (16):8#35V0
- U$122: device buzzard_labels (15):A#0 -> buzzard_labels (16):VIN1
- U$123: device buzzard_labels (15):A#1 -> buzzard_labels (16):E#STOP2
- U$124: device buzzard_labels (15):B#2 -> buzzard_labels (16):LIM_SW3
- U$125: device buzzard_labels (15):B#3 -> buzzard_labels (16):INT4
- U$126: device buzzard_labels (27):SERIAL0 -> buzzard_labels (18):ADR0
- U$127: device buzzard_labels (19):INT2 -> buzzard_labels (18):RESET1
- U$128: device buzzard_labels (19):GND1 -> SparkFun-Aesthetics:QWIIC_5.5MM
- U$129: device buzzard_labels (19):PWR0 -> buzzard_labels (16):INT4
- U$13: device buzzard_labels (16):VIN1 -> buzzard_labels (43):STAT0
- U$130: device buzzard_labels (8):3V30 -> buzzard_labels (19):3V35
- U$131: device buzzard_labels (8):3V37 -> buzzard_labels (19):GND6
- U$132: device buzzard_labels (8):GND8 -> buzzard_labels (19):SDA4
- U$133: device buzzard_labels (8):SCL5 -> buzzard_labels (19):SCL3
- U$134: device buzzard_labels (8):SDA6 -> buzzard_labels (19):INT2
- U$135: device buzzard_labels (8):STEP4 -> buzzard_labels (19):GND1
- U$136: device buzzard_labels (8):VIN3 -> buzzard_labels (19):PWR0
- U$137: device buzzard_labels (13):STAT5 -> buzzard_labels (28):3V31
- U$138: device buzzard_labels (15):A#0 -> buzzard_labels (28):STEP2
- U$139: device buzzard_labels (15):A#1 -> buzzard_labels (28):VIN0
- U$140: device buzzard_labels (15):B#2 -> buzzard_labels (34):QWIIC_STEP0
- U$141: device buzzard_labels (15):B#3 -> buzzard_labels (31):A#2
- U$142: device SparkX:SPARKX-MEDIUM -> buzzard_labels (31):A#3
- U$143: device buzzard_labels:BLK2 -> buzzard_labels (31):B#4
- U$144: device buzzard_labels:BLK2 -> buzzard_labels (31):B#5
- U$145: device buzzard_labels:GRN1 -> buzzard_labels (38):3V31
- U$146: device buzzard_labels:GRN1 -> buzzard_labels (38):DTR4
- U$147: device SparkFun-Aesthetics:QWIIC_5.5MM -> buzzard_labels (38):GND0
- U$148: device buzzard_labels (16):8#35V0 -> buzzard_labels (38):GND0
- U$149: device buzzard_labels (16):8#35V0 -> buzzard_labels (38):RXI3
- U$15: device buzzard_labels (15):A#0 -> Labels:I_SUPER2_C-()-03
- U$150: device buzzard_labels (16):VIN1 -> buzzard_labels (38):TXO2
- U$151: value (none) -> SPARKX-LOGO4; device buzzard_labels (16):VIN1 -> SparkX:SPARKX-MEDIUM
- U$152: device buzzard_labels (16):E#STOP2 -> buzzard_labels (39):DEBUG0
- U$153, U$67: device buzzard_labels (16):LIM_SW3 -> buzzard_labels (16):8#35V0
- U$154: device buzzard_labels (16):INT4 -> buzzard_labels (42):GND0
- U$155: device buzzard_labels (18):ADR0 -> buzzard_labels (42):PWR1
- U$156: device buzzard_labels (18):RESET1 -> buzzard_labels (42):A#2
- U$157: device SparkFun-Aesthetics:QWIIC_5.5MM -> buzzard_labels (42):A#3
- U$158: device buzzard_labels (16):INT4 -> buzzard_labels (42):B#4
- U$159: device buzzard_labels (25):QWIIC_STEP0 -> buzzard_labels (42):B#5
- U$16: device buzzard_labels (15):A#1 -> Labels:I_SUPER2_C-()-03
- U$160: device buzzard_labels (19):3V35 -> buzzard_labels (43):STAT0
- U$161: device buzzard_labels (19):GND6 -> Labels:I_SUPER2_C-()-03
- U$162: device buzzard_labels (19):SDA4 -> Labels:I_SUPER2_C-()-03
- U$163: device buzzard_labels (19):SCL3 -> buzzard_labels (8):3V30
- U$164: device buzzard_labels (26):PROG0 -> buzzard_labels (8):3V37
- U$165: device buzzard_labels (15):A#0 -> buzzard_labels (8):GND8
- U$166: device buzzard_labels (15):A#1 -> buzzard_labels (8):SCL5
- U$167: device buzzard_labels (15):B#2 -> buzzard_labels (8):SDA6
- U$168: device buzzard_labels (15):B#3 -> buzzard_labels (8):STEP4
- U$169: device buzzard_labels (27):SERIAL0 -> buzzard_labels (8):VIN3
- U$17: device buzzard_labels (15):B#2 -> buzzard_labels (38):3V31
- U$170: device buzzard_labels (19):INT2 -> buzzard_labels (13):STAT5
- U$171: device buzzard_labels (19):GND1 -> buzzard_labels:BLK2
- U$172: device buzzard_labels (19):PWR0 -> buzzard_labels:GRN1
- U$18: device buzzard_labels (15):B#3 -> buzzard_labels (38):DTR4
- U$19: device SparkX:SPARKX-MEDIUM -> buzzard_labels (39):DEBUG0
- U$21: device buzzard_labels:BLK2 -> buzzard_labels (38):GND0
- U$22: device buzzard_labels:GRN1 -> buzzard_labels (38):GND0
- U$32: device buzzard_labels (25):QWIIC_STEP0 -> buzzard_labels (31):A#2
- U$35: device buzzard_labels (26):PROG0 -> buzzard_labels (38):RXI3
- U$36: device buzzard_labels (15):A#0 -> buzzard_labels (31):A#3
- U$37: device buzzard_labels (15):A#1 -> buzzard_labels (28):STEP2
- U$38: device buzzard_labels (15):B#2 -> buzzard_labels (28):VIN0
- U$39: device buzzard_labels (15):B#3 -> buzzard_labels (8):3V30
- U$40: device buzzard_labels (27):SERIAL0 -> buzzard_labels (16):8#35V0
- U$44: device buzzard_labels (8):3V30 -> buzzard_labels (42):GND0
- U$45: device buzzard_labels (8):3V37 -> buzzard_labels (28):3V31
- U$46, U$89: device buzzard_labels (8):GND8 -> buzzard_labels (31):B#4
- U$47, U$90: device buzzard_labels (8):SCL5 -> buzzard_labels (31):B#5
- U$48: device buzzard_labels (8):SDA6 -> buzzard_labels (38):TXO2
- U$49: value (none) -> SPARKX-LOGO4; device buzzard_labels (8):STEP4 -> SparkX:SPARKX-MEDIUM
- U$50: device buzzard_labels (8):VIN3 -> buzzard_labels (8):3V37
- U$51: device buzzard_labels (13):STAT5 -> buzzard_labels (8):GND8
- U$52: device buzzard_labels (15):A#0 -> buzzard_labels (8):SCL5
- U$53: device buzzard_labels (15):A#1 -> buzzard_labels (42):PWR1
- U$54: device buzzard_labels (15):B#2 -> buzzard_labels (42):A#2
- U$55: device buzzard_labels (15):B#3 -> buzzard_labels (42):A#3
- U$56: device SparkX:SPARKX-MEDIUM -> buzzard_labels (34):QWIIC_STEP0
- U$57: device buzzard_labels:BLK2 -> buzzard_labels (42):B#4
- U$58: device buzzard_labels:BLK2 -> buzzard_labels (42):B#5
- U$59: device buzzard_labels:GRN1 -> buzzard_labels (8):SDA6
- U$60: device buzzard_labels:GRN1 -> buzzard_labels (8):STEP4
- U$61: device SparkFun-Aesthetics:QWIIC_5.5MM -> buzzard_labels (8):VIN3
- U$62: device buzzard_labels (16):8#35V0 -> buzzard_labels (13):STAT5
- U$63: device buzzard_labels (16):8#35V0 -> buzzard_labels:BLK2
- U$64: device buzzard_labels (16):VIN1 -> buzzard_labels:GRN1
- U$65: device buzzard_labels (16):VIN1 -> SparkFun-Aesthetics:QWIIC_5.5MM
- U$66: device buzzard_labels (16):E#STOP2 -> buzzard_labels (16):8#35V0
- U$68: device buzzard_labels (16):INT4 -> buzzard_labels (16):VIN1
- U$69: device buzzard_labels (18):ADR0 -> buzzard_labels (16):E#STOP2
- U$70: device buzzard_labels (18):RESET1 -> buzzard_labels (16):LIM_SW3
- U$71: device SparkFun-Aesthetics:QWIIC_5.5MM -> buzzard_labels (16):INT4
- U$72: device buzzard_labels (16):INT4 -> buzzard_labels (18):ADR0
- U$73: device buzzard_labels (25):QWIIC_STEP0 -> buzzard_labels (18):RESET1
- U$74: device buzzard_labels (19):3V35 -> SparkFun-Aesthetics:QWIIC_5.5MM
- U$75: device buzzard_labels (19):GND6 -> buzzard_labels (16):INT4
- U$76: device buzzard_labels (19):SDA4 -> buzzard_labels (19):3V35
- U$77: device buzzard_labels (19):SCL3 -> buzzard_labels (19):GND6
- U$78: device buzzard_labels (26):PROG0 -> buzzard_labels (19):SDA4
- U$79: device buzzard_labels (15):A#0 -> buzzard_labels (19):SCL3
- U$80: device buzzard_labels (15):A#1 -> buzzard_labels (19):INT2
- U$81: device buzzard_labels (15):B#2 -> buzzard_labels (19):GND1
- U$82: device buzzard_labels (15):B#3 -> buzzard_labels (19):PWR0
- U$83: device buzzard_labels (27):SERIAL0 -> buzzard_labels (28):3V31
- U$84: device buzzard_labels (19):INT2 -> buzzard_labels (28):STEP2
- U$85: device buzzard_labels (19):GND1 -> buzzard_labels (28):VIN0
- U$86: device buzzard_labels (19):PWR0 -> buzzard_labels (34):QWIIC_STEP0
- U$87: device buzzard_labels (8):3V30 -> buzzard_labels (31):A#2
- U$88: device buzzard_labels (8):3V37 -> buzzard_labels (31):A#3
- U$91: device buzzard_labels (8):SDA6 -> buzzard_labels (38):3V31
- U$92: device buzzard_labels (8):STEP4 -> buzzard_labels (38):DTR4
- U$93: device buzzard_labels (8):VIN3 -> buzzard_labels (38):GND0
- U$94: device buzzard_labels (13):STAT5 -> buzzard_labels (38):GND0
- U$95: device buzzard_labels (15):A#0 -> buzzard_labels (38):RXI3
- U$96: device buzzard_labels (15):A#1 -> buzzard_labels (38):TXO2
- U$97: value (none) -> SPARKX-LOGO4; device buzzard_labels (15):B#2 -> SparkX:SPARKX-MEDIUM
- U$98: device buzzard_labels (15):B#3 -> buzzard_labels (39):DEBUG0
- U$99: device SparkX:SPARKX-MEDIUM -> buzzard_labels (16):8#35V0
- U10, U7: value A4988ALT1 -> ATMEGA328P_TQFP; device SparkFun-IC-Special-Function:QFN-28-5MM -> SparkFun-IC-Microcontroller:TQFP32-08
- U11, U5, U8: value ATMEGA328P_TQFP -> OPA344; device SparkFun-IC-Microcontroller:TQFP32-08 -> SparkFun-IC-Amplifiers:SOT23-5
- U4: value HV7801 -> ATMEGA328P_TQFP; device SparkFun-IC-Special-Function:SOT23-5 -> SparkFun-IC-Microcontroller:TQFP32-08
- U6, U9: value HV7801 -> A4988ALT1; device SparkFun-IC-Special-Function:SOT23-5 -> SparkFun-IC-Special-Function:QFN-28-5MM
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Connections:
- removed net ADR: JP2.2, U2.15
- removed net ADR1: JP18.2, U5.15
- removed net ADR2: JP27.2, U8.15
- removed net ADR3: JP36.2, U11.15
- removed net CURR_SENSE: U2.19, U4.5
- removed net CURR_SENSE1: U5.19, U6.5
- removed net CURR_SENSE2: U8.19, U9.5
- removed net CURR_SENSE3: U11.19, U12.5
- removed net EP: U2.25
- removed net EP1: U5.25
- removed net EP2: U8.25
- removed net EP3: U11.25
- removed net MOTOR_SUPPLY: R6.2, U1.22, U1.28, U4.1
- removed net MOTOR_SUPPLY1: R28.2, U3.22, U3.28, U6.1
- removed net MOTOR_SUPPLY2: R42.2, U7.22, U7.28, U9.1
- removed net MOTOR_SUPPLY3: R56.2, U10.22, U10.28, U12.1
- removed net N$3 (its old number): R8.2, U3.23
- new net AMP_CUR_SENSE: R9.2, U2.19, U44.1
- new net AMP_CUR_SENSE1: R32.2, U4.19, U5.1
- new net AMP_CUR_SENSE2: R49.2, U7.19, U8.1
- new net AMP_CUR_SENSE3: R66.2, U10.19, U11.1
- new net CURRENT_SENSE: R18.2, U1.27, U44.3
- new net CURRENT_SENSE1: R13.2, U3.27, U5.3
- new net CURRENT_SENSE2: R35.2, U6.27, U8.3
- new net CURRENT_SENSE3: R52.2, U11.3, U9.27
- new net MOSI: J5.4, U2.15
- new net MOSI1: J16.4, U4.15
- new net MOSI2: J27.4, U7.15
- new net MOSI3: J38.4, U10.15
- new net N$32: R26.2, STEP1.1
- new net N$73: R58.2, VIN3.1
- new net N$74: D16.A, J34.VIN0, J43.P$1
- new net N$75: D17.A, R60.1
- new net N$76: R60.2, STEP3.1
- new net N$77: U10.7, Y4.1
- new net N$78: U10.8, Y4.3
- new net N$79: D18.A, R63.1
- new net N$80: 3V4.1, R63.2
- new net N$81: JP21.1, R59.2
- new net N$82: R65.1, R66.1, U11.4
- new net N$83: R53.2, U9.23
- new net N$84: ADR3.1, U10.22
- new net N$85: D19.A, R61.1
- new net N$86: JP24.3, R67.2
- new net N$87: JP24.1, R68.2
- new net N$88: R61.2, SCK3.1
- net !ENABLE!: no longer J5.4
- net !ENABLE!1: now also R23.1, U4.14; no longer J16.4, R17.1, U5.14
- net !ENABLE!2: now also R40.1, U6.2, U7.14; no longer J27.4, R34.1, U7.2, U8.14
- net !ENABLE!3: now also R57.1, U10.14, U9.2; no longer J38.4, R48.1, U10.2, U11.14
- net !RST!1: now also C25.2, R28.1, U4.29; no longer C24.2, R25.1, U5.29
- net !RST!2: now also C38.2, R45.1, U7.29; no longer C36.2, R39.1, U8.29
- net !RST!3: now also C51.2, R62.1, U10.29; no longer C48.2, R53.1, U11.29
- net !SLEEP!1: now also R21.1, U4.2; no longer R13.1, U5.2
- net !SLEEP!2: now also R38.1, U6.14, U7.2; no longer R32.1, U7.14, U8.2
- net !SLEEP!3: now also R55.1, U10.2, U9.14; no longer R46.1, U10.14, U11.2
- net 3.3V: now also 3V3.2, C12.1, JP1.2, U44.5; no longer JP13.2
- net 3.3V1: now also 3V1.2, C16.1, C23.1, C26.1, JP4.2, R21.2, R22.2, R23.2, R28.2, U4.18, U4.4, U4.6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; no longer C15.1, C22.1, JP17.2, R13.2, R16.2, R17.2, R25.2, U5.18, U5.4, U5.6
- net 3.3V2: now also 3V2.2, C29.1, C36.1, C39.1, JP15.2, JP18.2, R38.2, R40.2, R45.2, U6.15, U7.18, U7.4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; no longer C27.1, C34.1, JP22.2, JP26.2, R32.2, R33.2, R34.2, U7.15, U8.18, U8.4, U8.6
- net 3.3V3: now also 3V4.2, C42.1, C49.1, C52.1, JP21.2, JP24.2, R55.2, R56.2, R57.2, R62.2, U10.18, U10.4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; no longer C39.1, C46.1, JP31.2, JP35.2, R46.2, R47.2, R48.2, R53.2, U10.15, U11.18, U11.4, U11.6
- net A49885_!RESET!: now also U2.23; no longer U2.22
- net A49885_!RESET!1: now also R22.1, U4.23; no longer R16.1, U5.22
- net A49885_!RESET!2: now also R39.1, U6.12, U7.23; no longer R33.1, U7.12, U8.22
- net A49885_!RESET!3: now also R56.1, U10.23, U9.12; no longer R47.1, U10.12, U11.22
- net AREF1: now also C22.1, U4.20; no longer C21.1, U5.20
- net AREF2: now also C35.1, U7.20; no longer C33.1, U8.20
- net AREF3: now also C48.1, U10.20; no longer C45.1, U11.20
- net COILA+: now also J6.P$4; no longer J6.4
- net COILA+1: now also J22.P$4; no longer J22.4
- net COILA+2: now also J33.P$4, U6.21; no longer J33.4, U7.21
- net COILA+3: now also J44.P$4, U9.21; no longer J44.4, U10.21
- net COILA-: now also J6.P$3; no longer J6.3
- net COILA-1: now also J22.P$3; no longer J22.3
- net COILA-2: now also J33.P$3, U6.24; no longer J33.3, U7.24
- net COILA-3: now also J44.P$3, U9.24; no longer J44.3, U10.24
- net COILB+: now also J6.P$1; no longer J6.1
- net COILB+1: now also J22.P$1; no longer J22.1
- net COILB+2: now also J33.P$1, U6.1; no longer J33.1, U7.1
- net COILB+3: now also J44.P$1, U9.1; no longer J44.1, U10.1
- net COILB-: now also J6.P$2; no longer J6.2
- net COILB-1: now also J22.P$2; no longer J22.2
- net COILB-2: now also J33.P$2, U6.26; no longer J33.2, U7.26
- net COILB-3: now also J44.P$2, U9.26; no longer J44.2, U10.26
- net CUR_REF1: now also C24.1, R30.2; no longer C23.1, R27.2
- net CUR_REF2: now also C37.1, R47.2, U6.17; no longer C35.1, R41.2, U7.17
- net CUR_REF3: now also C50.1, R64.2, U9.17; no longer C47.1, R55.2, U10.17
- net CUR_REF_PWM1: now also R30.1, U4.9; no longer R27.1, U5.9
- net CUR_REF_PWM2: now also R47.1, U7.9; no longer R41.1, U8.9
- net CUR_REF_PWM3: now also R64.1, U10.9; no longer R55.1, U11.9
- net DIR1: now also U4.10; no longer U5.10
- net DIR2: now also U6.19, U7.10; no longer U7.19, U8.10
- net DIR3: now also U10.10, U9.19; no longer U10.19, U11.10
- net DTR1: now also C25.1; no longer C24.1
- net DTR2: now also C38.1; no longer C36.1
- net DTR3: now also C51.1; no longer C48.1
- net GND: now also ADR.2, C12.2, J9.P$2, R7.2, U44.2; no longer J9.2, JP2.1, U4.4
- net GND1: now also ADR1.2, C13.2, C19.2, C21.-, C24.2, C26.2, J21.P$2, R13.1, R16.1, R17.2, R31.2, U4.21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; no longer C12.2, C15.2, C20.-, C21.2, J21.2, JP18.1, R7.1, R8.1, R9.2, U5.21, U5.3, U5.5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
- net GND2: now also ADR2.2, C31.2, C32.2, C34.-, C36.2, C37.2, C39.2, J32.P$2, R35.1, R36.1, R37.2, R48.2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; no longer C25.2, C28.2, C32.-, C33.2, C34.2, J32.2, JP27.1, R29.1, R30.1, R31.2, U7.18, U7.29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
- net GND3: now also ADR3.2, C43.2, C44.2, C47.-, C48.2, C49.2, C50.2, C52.2, J43.P$2, R52.1, R53.1, R54.2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; no longer C37.2, C39.2, C41.2, C44.-, C46.2, C47.2, J43.2, JP36.1, R43.1, R44.1, R45.2, U10.18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
- net INT10: now also U10.1; no longer U11.1
- net INT2: now also R25.1, U4.24; no longer R22.1, U5.24
- net INT3: now also U4.32; no longer U5.32
- net INT4: now also U4.1; no longer U5.1
- net INT5: now also R42.1, U7.24; no longer R36.1, U8.24
- net INT6: now also U7.32; no longer U8.32
- net INT7: now also U7.1; no longer U8.1
- net INT8: now also R59.1, U10.24; no longer R50.1, U11.24
- net INT9: now also U10.32; no longer U11.32
- net MISO1: now also U4.16; no longer U5.16
- net MISO2: now also U7.16; no longer U8.16
- net MISO3: now also U10.16; no longer U11.16
- net MS10: now also U10.12, U9.10; no longer U10.10, U11.12
- net MS11: now also U9.11; no longer U11.11
- net MS12: now also U10.13, U9.9; no longer U10.9, U11.13
- net MS4: now also U4.12; no longer U5.12
- net MS5: now also U4.11; no longer U5.11
- net MS6: now also U4.13; no longer U5.13
- net MS7: now also U6.10, U7.12; no longer U7.10, U8.12
- net MS8: now also U6.11; no longer U8.11
- net MS9: now also U6.9, U7.13; no longer U7.9, U8.13
- net N$11: now also STEP.1; no longer JP11.1
- net N$12: now also R12.1; no longer R12.2
- net N$15: now also JP1.3, R6.2; no longer C13.2, U3.5
- net N$16: now also JP1.1, R8.2; no longer R9.1, U3.13
- net N$17: now also R12.2, SCK.1; no longer C18.1, U3.8
- net N$18: now also C15.1, U3.4; no longer C19.1, U3.6
- net N$2: now also R7.1, R9.1, U44.4; no longer R7.2, U3.27
- net N$22: now also C15.2, U3.5; no longer D10.A, R21.1
- net N$23: now also R17.1, U3.13; no longer JP5.1, R21.2
- net N$24: now also C19.1, U3.8; no longer D6.A, J12.VIN0, J21.1
- net N$25: now also C20.1, U3.6; no longer D7.A, R23.1
- net N$27: now also 3V3.1; no longer JP13.1
- net N$28: now also D10.A, R24.1; no longer JP16.1, R23.2
- net N$29: now also VIN1.1; no longer D9.A
- net N$30: now also D6.A, J12.VIN0, J21.P$1; no longer U5.7, Y2.1
- net N$31: now also D7.A, R26.1; no longer R18.2, U1.27
- net N$33: now also U4.7, Y2.1; no longer U5.8, Y2.3
- net N$34: now also U4.8, Y2.3; no longer D8.A, R26.1
- net N$35: now also D8.A, R29.1; no longer JP17.1, R26.2
- net N$36: now also 3V1.1, R29.2; no longer JP12.1, R22.2
- net N$37: now also JP4.1, R25.2; no longer R29.2, U7.27
- net N$38: now also R31.1, R32.1, U5.4; no longer R30.2, U7.23
- net N$39: now also R16.2, U3.23; no longer C26.1, U7.4
- net N$4: now also VIN.1; no longer JP1.1
- net N$40: now also ADR1.1, U4.22; no longer C26.2, U7.5
- net N$41: now also D9.A, R27.1; no longer R31.1, U7.13
- net N$42: now also JP12.3, R33.2; no longer C30.1, U7.8
- net N$43: now also JP12.1, R34.2; no longer C31.1, U7.6
- net N$44: now also R27.2, SCK1.1; no longer D15.A, R35.1
- net N$45: now also C28.1, U6.4; no longer JP21.1, R35.2
- net N$46: now also C28.2, U6.5; no longer D11.A, J23.VIN0, J32.1
- net N$47: now also U6.13; no longer D12.A
- net N$48: now also C32.1, U6.8; no longer JP25.1, R37.2
- net N$49: now also C33.1, U6.6; no longer D14.A, R38.2
- net N$50: now also D15.A, R41.1; no longer U8.7, Y3.1
- net N$51: now also R41.2, VIN2.1; no longer U8.8, Y3.3
- net N$52: now also D11.A, J23.VIN0, J32.P$1; no longer D13.A, R40.1
- net N$53: now also D12.A, R43.1; no longer JP26.1, R40.2
- net N$54: now also R43.2, STEP2.1; no longer JP22.1, R36.2
- net N$55: now also U7.7, Y3.1; no longer R43.2, U10.27
- net N$56: now also U7.8, Y3.3; no longer R44.2, U10.23
- net N$57: now also D13.A, R46.1; no longer C38.1, U10.4
- net N$58: now also 3V2.1, R46.2; no longer C38.2, U10.5
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Routing:
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- added copper zone on layer 2, net 3.3V
- added copper zone on layer 2, net 3.3V1
- added copper zone on layer 2, net 3.3V2
- added copper zone on layer 2, net 3.3V3
- added copper zone on layer 1, net CURRENT_SENSE
- added copper zone on layer 1, net CURRENT_SENSE1
- added copper zone on layer 1, net CURRENT_SENSE2
- added copper zone on layer 1, net CURRENT_SENSE3
- added copper zone on layer 15, net GND
- added copper zone on layer 15, net GND1
- added copper zone on layer 15, net GND2
- added copper zone on layer 15, net GND3
- added copper zone on layer 1, net N$39
- added copper zone on layer 1, net N$61
- added copper zone on layer 1, net N$83
- added copper zone on layer 1, net VIN
- added copper zone on layer 2, net VIN
- added copper zone on layer 1, net VIN1
- added copper zone on layer 2, net VIN1
- added copper zone on layer 1, net VIN2
- added copper zone on layer 2, net VIN2
- added copper zone on layer 1, net VIN3
- added copper zone on layer 2, net VIN3
- removed copper zone on layer 1, net MOTOR_SUPPLY
- removed copper zone on layer 1, net MOTOR_SUPPLY1
- removed copper zone on layer 1, net MOTOR_SUPPLY2
- removed copper zone on layer 1, net MOTOR_SUPPLY3
- removed copper zone on layer 1, net N$2
- removed copper zone on layer 1, net N$3 (its old number)
- removed copper zone on layer 1, net N$31
- removed copper zone on layer 1, net N$37
- removed copper zone on layer 1, net N$38
- removed copper zone on layer 1, net N$55
- removed copper zone on layer 1, net N$56
